File: hardware/boards/high-power/bms.kicad_sch (KiCad schematic)
At the start: 31 parts, among them J2 Cell Taps, J3 10k NTC Thermistor, J4 10k NTC Thermistor, Q1 HYG009N04LS1C2, Q2 HYG009N04LS1C2, U1 MAX17320G20+T

Commit message: Add initial changes after schematic review
Parts:
- R202: renamed from R2; value 19R 1/2W -> 27R 1/2W
- R203: renamed from R3; value 19R 1/2W -> 27R 1/2W
- R204: renamed from R4; value 19R 1/2W -> 27R 1/2W
- R205: renamed from R5; value 38R 1/2W -> 51R 1/2W
- renumbered BT1 to BT201, C1 to C201, C2 to C202, C3 to C203, C4 to C204, C5 to C205, C6 to C206, C7 to C207, C8 to C208, C9 to C209, C10 to C210, F1 to F201, J2 to J201, J3 to J202, J4 to J203, Q1 to Q201, Q2 to Q202, R1 to R201, R6 to R206, R7 to R207, R8 to R208, R9 to R209, R10 to R210, R11 to R211, TP1 to TP201, TP2 to TP202, U1 to U201
Connections:
- net at Q201.2 (G), R208.1: now also C207.2
- net at J202.1 (Pin_1): now also U201.16 (TH2); no longer U201.19 (TH4)
- net at U201.10 (TH1): now also J203.1 (Pin_1)
- net at U201.18 (TH3): no longer J203.1 (Pin_1)
- net at R208.2, U201.3 (CHG): no longer C207.2
- no-connect marks 3 -> 1
Other:
- moved on the sheet: C207, J202, J203, R208, R209
