File: hardware/boards/high-power/charge_controller.kicad_sch (KiCad schematic)
At the start: 64 parts, among them Q10 DMN3020UFDF-7, Q11 AONR21321, Q6 SSM3J35AMFV,L3F, Q7 DMN3020UFDF-7, Q8 DMN3020UFDF-7, Q9 DMN3020UFDF-7, U3 MCP47A1T, U4 BQ25703ARSNT

Commit message: Add initial changes after schematic review
Parts:
- removed Q6: SSM3J35AMFV,L3F, symbol Device:Q_PMOS_DGS
- removed R21: 10k, symbol Device:R
- removed R26: 100, symbol Device:R
- removed R31: 50R, symbol Device:R
- removed TP6: ILIM_HIZ, symbol Connector:TestPoint
- removed U3: MCP47A1T, symbol power_and_charging:MCP47A1T
- added C429: 1nF, symbol Device:C_Small
- added R413, R414: 0R, symbol Device:R
- R410: renamed from R25; value 320 -> 10k
- renumbered C27 to C401, C28 to C402, C29 to C403, C30 to C404, C31 to C405, C32 to C406, C33 to C407, C34 to C408, C35 to C409, C36 to C410, C37 to C411, C38 to C412, C39 to C413, C40 to C414, C41 to C415, C42 to C416, C43 to C417, C44 to C418, C45 to C419, C46 to C420, C47 to C421, C48 to C422, C49 to C423, C50 to C424, C51 to C425, C52 to C426, C53 to C427, C54 to C428, L2 to L401, Q7 to Q401, Q8 to Q402, Q9 to Q403, Q10 to Q404, Q11 to Q405, R19 to R401, R20 to R402, R22 to R403, R23 to R404, R24 to R405, R27 to R406, R28 to R407, R29 to R408, R30 to R409, R32 to R411, R33 to R412, R34 to R415, R35 to R416, R36 to R417, R37 to R418, R38 to R419, R39 to R420, R40 to R421, R41 to R422, TP7 to TP401, TP8 to TP402, TP9 to TP403, U4 to U401
Connections:
- net +3V3: now also R410.2
- net GND: now also C429.2, R413.2, R414.2; no longer U401.14 (CMPIN), U401.5 (EN_OTG)
- net REGN: no longer R410.1
- net ~{PROCHOT}: now also R410.1
- net at C414.1, Q401.1 (D), R405.2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: now also C429.1
- new net: R413.1, U401.5 (EN_OTG)
- new net: R414.1, U401.14 (CMPIN)
Other:
- note added: "8A INDUCTOR SATURATION CURRENT"
- note removed: "Check this pullup to 1.05V. ~{PROCHOT} apparently draws 5mA"
- moved on the sheet: C414, R410, R415
