File: hardware/boards/high-power/esc.kicad_sch (KiCad schematic)
At the start: 70 parts, among them Q19 Q_NMOS_DGS, Q20 Q_NMOS_DGS, Q21 Q_NMOS_DGS, Q22 Q_NMOS_DGS, Q23 Q_NMOS_DGS, Q24 Q_NMOS_DGS, U9 MCT8329A

Commit message: Add initial changes after schematic review
Parts:
- R803: renamed from R90; value 100k -> 10k
- R804: renamed from R91; value 100k -> 10k
- renumbered C83 to C801, C84 to C802, C85 to C803, C86 to C804, C87 to C805, C88 to C806, C89 to C807, C90 to C808, C91 to C809, C92 to C810, C93 to C811, C94 to C812, C95 to C813, C96 to C814, C97 to C815, C98 to C816, C99 to C817, C100 to C818, C101 to C819, C102 to C820, C103 to C821, C104 to C822, D11 to D801, D12 to D802, D13 to D803, D14 to D804, D15 to D805, D16 to D806, D17 to D807, D18 to D808, D19 to D809, Q19 to Q801, Q20 to Q802, Q21 to Q803, Q22 to Q804, Q23 to Q805, Q24 to Q806, R88 to R801, R89 to R802, R92 to R805, R93 to R806, R94 to R807, R95 to R808, R96 to R809, R97 to R810, R98 to R811, R99 to R812, R100 to R813, R101 to R814, R102 to R815, R103 to R816, R104 to R817, R105 to R818, R106 to R819, R107 to R820, R108 to R821, R109 to R822, R110 to R823, R111 to R824, R112 to R825, R113 to R826, R114 to R827, R115 to R828, R116 to R829, R117 to R830, R118 to R831, R119 to R832, U9 to U801
Connections:
- net +3V3: no longer C801.2, C802.2, R807.2, U801.26 (AVDD)
- net GND: now also C802.2; no longer C802.1
- net at R807.1: now also C801.2, U801.26 (AVDD); no longer U801.2 (VREG)
- new net: C802.1, R807.2, U801.2 (VREG)
Other:
- moved on the sheet: C801, C802, R807
