File: hardware/boards/high-power/high-power.kicad_sch (KiCad schematic)
At the start: 1 part, among them J5 Conn_01x32_Pin

Commit message: Add initial changes after schematic review
Parts:
- renumbered J5 to J101
Changed lines of the file:
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@@
   (symbol (lib_id "power:+BATT") (at 116.84 113.665 270) (unit 1)
     (in_bom yes) (on_board yes) (dnp no)
-    (property "Reference" "#PWR0153" (at 113.03 113.665 0)
+    (property "Reference" "#PWR0103" (at 113.03 113.665 0)
       (effects (font (size 1.27 1.27)) hide)
     )
@@
       (project "high-power"
         (path "/4aa4a0cf-3721-431d-88e8-8afb2cf87302"
-          (reference "#PWR0153") (unit 1)
+          (reference "#PWR0103") (unit 1)
         )
       )
@@
   (symbol (lib_id "power:+5V") (at 116.84 111.125 270) (unit 1)
     (in_bom yes) (on_board yes) (dnp no)
-    (property "Reference" "#PWR02" (at 113.03 111.125 0)
+    (property "Reference" "#PWR0102" (at 113.03 111.125 0)
       (effects (font (size 1.27 1.27)) hide)
     )
@@
       (project "high-power"
         (path "/4aa4a0cf-3721-431d-88e8-8afb2cf87302"
-          (reference "#PWR02") (unit 1)
+          (reference "#PWR0102") (unit 1)
         )
       )
@@
   (symbol (lib_id "power:+3.3V") (at 116.84 108.585 270) (unit 1)
     (in_bom yes) (on_board yes) (dnp no)
-    (property "Reference" "#PWR01" (at 113.03 108.585 0)
+    (property "Reference" "#PWR0101" (at 113.03 108.585 0)
       (effects (font (size 1.27 1.27)) hide)
     )
@@
       (project "high-power"
         (path "/4aa4a0cf-3721-431d-88e8-8afb2cf87302"
-          (reference "#PWR01") (unit 1)
+          (reference "#PWR0101") (unit 1)
         )
       )
@@
   (symbol (lib_id "Connector:Conn_01x32_Pin") (at 109.855 111.125 0) (unit 1)
     (in_bom yes) (on_board yes) (dnp no) (fields_autoplaced)
-    (property "Reference" "J5" (at 110.49 69.215 0)
+    (property "Reference" "J101" (at 110.49 69.215 0)
       (effects (font (size 1.27 1.27)))
     )
@@
       (project "high-power"
         (path "/4aa4a0cf-3721-431d-88e8-8afb2cf87302"
-          (reference "J5") (unit 1)
+          (reference "J101") (unit 1)
         )
       )
@@
   (symbol (lib_id "power:GND") (at 116.84 153.035 0) (unit 1)
     (in_bom yes) (on_board yes) (dnp no) (fields_autoplaced)
-    (property "Reference" "#PWR0154" (at 116.84 159.385 0)
+    (property "Reference" "#PWR0104" (at 116.84 159.385 0)
       (effects (font (size 1.27 1.27)) hide)
     )
@@
       (project "high-power"
         (path "/4aa4a0cf-3721-431d-88e8-8afb2cf87302"
-          (reference "#PWR0154") (unit 1)
+          (reference "#PWR0104") (unit 1)
         )
       )
