File: hardware/boards/high-power/hotswap.kicad_sch (KiCad schematic)
At the start: 20 parts, among them Q12 HYG009N04LS1C2, SW1 SW_SPDT, U5 LT1641-1

Commit message: Add initial changes after schematic review
Parts:
- renumbered C55 to C501, C56 to C502, C57 to C503, C58 to C504, D1 to D501, Q12 to Q501, R42 to R501, R43 to R502, R44 to R503, R45 to R504, R46 to R505, R47 to R506, R48 to R507, R49 to R508, R50 to R509, R51 to R510, R52 to R511, SW1 to SW501, TP10 to TP501, U5 to U501
