File: hardware/boards/high-power/motors.kicad_sch (KiCad schematic)
At the start: 7 parts, among them U6 TCA9539RTWR, U7 LM75BTP,147

Commit message: Add initial changes after schematic review
Parts:
- renumbered C59 to C601, C60 to C602, R53 to R601, R54 to R602, R55 to R603, U6 to U601, U7 to U602
Changed lines of the file:
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@@
   (symbol (lib_id "Device:C") (at 140.335 165.735 0) (unit 1)
     (in_bom yes) (on_board yes) (dnp no)
-    (property "Reference" "C60" (at 142.875 165.1 0)
+    (property "Reference" "C602" (at 142.875 165.1 0)
       (effects (font (size 1.27 1.27)) (justify left))
     )
@@
       (project "high-power"
         (path "/4aa4a0cf-3721-431d-88e8-8afb2cf87302/808c67f5-175b-4ddf-aa25-2f2591470087"
-          (reference "C60") (unit 1)
+          (reference "C602") (unit 1)
         )
         (path "/4aa4a0cf-3721-431d-88e8-8afb2cf87302"
@@
   (symbol (lib_id "power:+3V3") (at 125.73 148.59 0) (unit 1)
     (in_bom yes) (on_board yes) (dnp no)
-    (property "Reference" "#PWR066" (at 125.73 152.4 0)
+    (property "Reference" "#PWR0604" (at 125.73 152.4 0)
       (effects (font (size 1.27 1.27)) hide)
     )
@@
       (project "high-power"
         (path "/4aa4a0cf-3721-431d-88e8-8afb2cf87302/808c67f5-175b-4ddf-aa25-2f2591470087"
-          (reference "#PWR066") (unit 1)
+          (reference "#PWR0604") (unit 1)
         )
         (path "/4aa4a0cf-3721-431d-88e8-8afb2cf87302"
@@
   (symbol (lib_id "Device:R") (at 107.315 67.31 0) (unit 1)
     (in_bom yes) (on_board yes) (dnp no)
-    (property "Reference" "R54" (at 109.22 66.675 0)
+    (property "Reference" "R602" (at 109.22 66.675 0)
       (effects (font (size 1.27 1.27)) (justify left))
     )
@@
       (project "high-power"
         (path "/4aa4a0cf-3721-431d-88e8-8afb2cf87302/808c67f5-175b-4ddf-aa25-2f2591470087"
-          (reference "R54") (unit 1)
+          (reference "R602") (unit 1)
         )
       )
@@
   (symbol (lib_id "power:GND") (at 90.17 64.77 0) (unit 1)
     (in_bom yes) (on_board yes) (dnp no) (fields_autoplaced)
-    (property "Reference" "#PWR063" (at 90.17 71.12 0)
+    (property "Reference" "#PWR0601" (at 90.17 71.12 0)
       (effects (font (size 1.27 1.27)) hide)
     )
@@
       (project "high-power"
         (path "/4aa4a0cf-3721-431d-88e8-8afb2cf87302/808c67f5-175b-4ddf-aa25-2f2591470087"
-          (reference "#PWR063") (unit 1)
+          (reference "#PWR0601") (unit 1)
         )
       )
@@
   (symbol (lib_id "Device:R") (at 113.03 154.94 0) (unit 1)
     (in_bom yes) (on_board yes) (dnp no)
-    (property "Reference" "R55" (at 114.935 153.67 0)
+    (property "Reference" "R603" (at 114.935 153.67 0)
       (effects (font (size 1.27 1.27)) (justify left))
     )
@@
       (project "high-power"
         (path "/4aa4a0cf-3721-431d-88e8-8afb2cf87302/808c67f5-175b-4ddf-aa25-2f2591470087"
-          (reference "R55") (unit 1)
+          (reference "R603") (unit 1)
         )
         (path "/4aa4a0cf-3721-431d-88e8-8afb2cf87302"
@@
   (symbol (lib_id "Device:R") (at 103.505 103.505 0) (unit 1)
     (in_bom yes) (on_board yes) (dnp no)
-    (property "Reference" "R53" (at 105.41 102.87 0)
+    (property "Reference" "R601" (at 105.41 102.87 0)
       (effects (font (size 1.27 1.27)) (justify left))
     )
@@
       (project "high-power"
         (path "/4aa4a0cf-3721-431d-88e8-8afb2cf87302/808c67f5-175b-4ddf-aa25-2f2591470087"
-          (reference "R53") (unit 1)
+          (reference "R601") (unit 1)
         )
       )
@@
   (symbol (lib_id "Capstone:TCA9539RTWR_") (at 125.095 85.725 0) (unit 1)
     (in_bom yes) (on_board yes) (dnp no)
-    (property "Reference" "U6" (at 128.27 60.96 0)
+    (property "Reference" "U601" (at 128.27 60.96 0)
       (effects (font (size 1.27 1.27)) (justify left))
     )
@@
       (project "high-power"
         (path "/4aa4a0cf-3721-431d-88e8-8afb2cf87302/808c67f5-175b-4ddf-aa25-2f2591470087"
-          (reference "U6") (unit 1)
+          (reference "U601") (unit 1)
         )
       )
@@
   (symbol (lib_id "power:GND") (at 125.095 114.3 0) (unit 1)
     (in_bom yes) (on_board yes) (dnp no) (fields_autoplaced)
-    (property "Reference" "#PWR065" (at 125.095 120.65 0)
+    (property "Reference" "#PWR0603" (at 125.095 120.65 0)
       (effects (font (size 1.27 1.27)) hide)
     )
@@
       (project "high-power"
         (path "/4aa4a0cf-3721-431d-88e8-8afb2cf87302/808c67f5-175b-4ddf-aa25-2f2591470087"
-          (reference "#PWR065") (unit 1)
+          (reference "#PWR0603") (unit 1)
         )
       )
@@
   (symbol (lib_id "Capstone:LM75BTP,147") (at 125.73 162.56 0) (unit 1)
     (in_bom yes) (on_board yes) (dnp no)
-    (property "Reference" "U7" (at 127.635 170.18 0)
+    (property "Reference" "U602" (at 127.635 170.18 0)
       (effects (font (size 1.27 1.27)) (justify left))
     )
@@
       (project "high-power"
         (path "/4aa4a0cf-3721-431d-88e8-8afb2cf87302/808c67f5-175b-4ddf-aa25-2f2591470087"
-          (reference "U7") (unit 1)
+          (reference "U602") (unit 1)
         )
         (path "/4aa4a0cf-3721-431d-88e8-8afb2cf87302"
@@
   (symbol (lib_id "power:+3V3") (at 125.095 57.785 0) (unit 1)
     (in_bom yes) (on_board yes) (dnp no)
-    (property "Reference" "#PWR064" (at 125.095 61.595 0)
+    (property "Reference" "#PWR0602" (at 125.095 61.595 0)
       (effects (font (size 1.27 1.27)) hide)
     )
@@
       (project "high-power"
         (path "/4aa4a0cf-3721-431d-88e8-8afb2cf87302/808c67f5-175b-4ddf-aa25-2f2591470087"
-          (reference "#PWR064") (unit 1)
+          (reference "#PWR0602") (unit 1)
         )
       )
@@
   (symbol (lib_id "Device:C") (at 98.425 59.055 270) (unit 1)
     (in_bom yes) (on_board yes) (dnp no)
-    (property "Reference" "C59" (at 96.52 55.88 90)
+    (property "Reference" "C601" (at 96.52 55.88 90)
       (effects (font (size 1.27 1.27)) (justify left))
     )
@@
       (project "high-power"
         (path "/4aa4a0cf-3721-431d-88e8-8afb2cf87302/808c67f5-175b-4ddf-aa25-2f2591470087"
-          (reference "C59") (unit 1)
+          (reference "C601") (unit 1)
         )
       )
@@
   (symbol (lib_id "power:GND") (at 125.73 173.99 0) (unit 1)
     (in_bom yes) (on_board yes) (dnp no) (fields_autoplaced)
-    (property "Reference" "#PWR067" (at 125.73 180.34 0)
+    (property "Reference" "#PWR0605" (at 125.73 180.34 0)
       (effects (font (size 1.27 1.27)) hide)
     )
@@
       (project "high-power"
         (path "/4aa4a0cf-3721-431d-88e8-8afb2cf87302/808c67f5-175b-4ddf-aa25-2f2591470087"
-          (reference "#PWR067") (unit 1)
+          (reference "#PWR0605") (unit 1)
         )
         (path "/4aa4a0cf-3721-431d-88e8-8afb2cf87302"
