File: hardware/boards/high-power/power_charging.kicad_sch (KiCad schematic)
At the start: 14 parts, among them Q25 Q_NMOS_DGS, U12 SLG55021, U13 SLG55021, U2 TCA9539RTWR

Commit message: Add initial changes after schematic review
Parts:
- added J1101: Conn_01x02_Pin, symbol Connector:Conn_01x02_Pin
- renumbered C149 to C1101, C150 to C1102, R184 to R1101, R185 to R1102, U12 to U1101, U13 to U1102
Connections:
- net at U2.16 (P16): now also J1101.2 (Pin_2)
- net at U2.17 (P17): now also J1101.1 (Pin_1)
- no-connect marks 2 -> 0
Changed lines of the file:
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@@
   (junction (at 71.12 84.455) (diameter 0) (color 0 0 0 0)
   )
-  (no_connect (at 210.82 120.015))
-  (no_connect (at 210.82 122.555))
   (wire (pts (xy 60.96 106.68) (xy 60.96 107.95))
     (stroke (width 0) (type default))
@@
         )
         (path "/4aa4a0cf-3721-431d-88e8-8afb2cf87302/e67f9728-ca0e-433d-883c-80e42a6fd80b"
-          (reference "#PWR0148") (unit 1)
+          (reference "#PWR01105") (unit 1)
         )
       )
@@
   (symbol (lib_name "GND_1") (lib_id "power:GND") (at 71.12 109.22 0) (unit 1)
     (in_bom yes) (on_board yes) (dnp no) (fields_autoplaced)
-    (property "Reference" "#PWR0145" (at 71.12 115.57 0)
+    (property "Reference" "#PWR01102" (at 71.12 115.57 0)
       (effects (font (size 1.27 1.27)) hide)
     )
@@
       (project "high-power"
         (path "/4aa4a0cf-3721-431d-88e8-8afb2cf87302/e67f9728-ca0e-433d-883c-80e42a6fd80b"
-          (reference "#PWR0145") (unit 1)
+          (reference "#PWR01102") (unit 1)
         )
       )
@@
         )
         (path "/4aa4a0cf-3721-431d-88e8-8afb2cf87302/e67f9728-ca0e-433d-883c-80e42a6fd80b"
-          (reference "#PWR0149") (unit 1)
+          (reference "#PWR01106") (unit 1)
         )
       )
@@
   (symbol (lib_id "Device:C") (at 97.155 102.87 0) (unit 1)
     (in_bom yes) (on_board yes) (dnp no)
-    (property "Reference" "C150" (at 100.33 101.6 0)
+    (property "Reference" "C1102" (at 100.33 101.6 0)
       (effects (font (size 1.27 1.27)) (justify left))
     )
@@
       (project "high-power"
         (path "/4aa4a0cf-3721-431d-88e8-8afb2cf87302/e67f9728-ca0e-433d-883c-80e42a6fd80b"
-          (reference "C150") (unit 1)
+          (reference "C1102") (unit 1)
         )
       )
@@
         )
         (path "/4aa4a0cf-3721-431d-88e8-8afb2cf87302/e67f9728-ca0e-433d-883c-80e42a6fd80b"
-          (reference "C151") (unit 1)
+          (reference "C1103") (unit 1)
         )
       )
@@
         )
         (path "/4aa4a0cf-3721-431d-88e8-8afb2cf87302/e67f9728-ca0e-433d-883c-80e42a6fd80b"
-          (reference "Q37") (unit 1)
+          (reference "Q1101") (unit 1)
         )
       )
@@
         )
         (path "/4aa4a0cf-3721-431d-88e8-8afb2cf87302/e67f9728-ca0e-433d-883c-80e42a6fd80b"
-          (reference "R186") (unit 1)
+          (reference "R1103") (unit 1)
         )
       )
@@
         )
         (path "/4aa4a0cf-3721-431d-88e8-8afb2cf87302/e67f9728-ca0e-433d-883c-80e42a6fd80b"
-          (reference "#PWR0150") (unit 1)
+          (reference "#PWR01107") (unit 1)
         )
       )
@@
         )
         (path "/4aa4a0cf-3721-431d-88e8-8afb2cf87302/e67f9728-ca0e-433d-883c-80e42a6fd80b"
-          (reference "U14") (unit 1)
+          (reference "U1103") (unit 1)
         )
       )
@@
         )
         (path "/4aa4a0cf-3721-431d-88e8-8afb2cf87302/e67f9728-ca0e-433d-883c-80e42a6fd80b"
-          (reference "TP12") (unit 1)
+          (reference "TP1102") (unit 1)
         )
       )
@@
     )
   )
+  (symbol (lib_id "Connector:Conn_01x02_Pin") (at 215.9 122.555 180) (unit 1)
+    (in_bom yes) (on_board yes) (dnp no) (fields_autoplaced)
+    (property "Reference" "J1101" (at 217.17 120.65 0)
+      (effects (font (size 1.27 1.27)) (justify right))
+    )
+    (property "Value" "Conn_01x02_Pin" (at 217.17 123.19 0)
+      (effects (font (size 1.27 1.27)) (justify right))
+    )
+    (property "Footprint" "" (at 215.9 122.555 0)
+      (effects (font (size 1.27 1.27)) hide)
+    )
+    (property "Datasheet" "~" (at 215.9 122.555 0)
+      (effects (font (size 1.27 1.27)) hide)
+    )
+    (pin "1")
+    (pin "2")
+    (instances
+      (project "high-power"
+        (path "/4aa4a0cf-3721-431d-88e8-8afb2cf87302/e67f9728-ca0e-433d-883c-80e42a6fd80b"
+          (reference "J1101") (unit 1)
+        )
+      )
+    )
+  )
   (symbol (lib_id "power:+5V") (at 71.12 83.185 0) (unit 1)
     (in_bom yes) (on_board yes) (dnp no) (fields_autoplaced)
-    (property "Reference" "#PWR0144" (at 71.12 86.995 0)
+    (property "Reference" "#PWR01101" (at 71.12 86.995 0)
       (effects (font (size 1.27 1.27)) hide)
     )
@@
       (project "high-power"
         (path "/4aa4a0cf-3721-431d-88e8-8afb2cf87302/e67f9728-ca0e-433d-883c-80e42a6fd80b"
-          (reference "#PWR0144") (unit 1)
+          (reference "#PWR01101") (unit 1)
         )
       )
@@
   (symbol (lib_id "capstone:SLG55021") (at 77.47 98.425 0) (unit 1)
     (in_bom yes) (on_board yes) (dnp no) (fields_autoplaced)
-    (property "Reference" "U12" (at 73.0759 84.455 0)
+    (property "Reference" "U1101" (at 73.0759 84.455 0)
       (effects (font (size 1.27 1.27)) (justify left))
     )
@@
       (project "high-power"
         (path "/4aa4a0cf-3721-431d-88e8-8afb2cf87302/e67f9728-ca0e-433d-883c-80e42a6fd80b"
-          (reference "U12") (unit 1)
+          (reference "U1101") (unit 1)
         )
       )
@@
   (symbol (lib_id "power:+5V") (at 120.015 83.185 0) (unit 1)
     (in_bom yes) (on_board yes) (dnp no) (fields_autoplaced)
-    (property "Reference" "#PWR0146" (at 120.015 86.995 0)
+    (property "Reference" "#PWR01103" (at 120.015 86.995 0)
       (effects (font (size 1.27 1.27)) hide)
     )
@@
       (project "high-power"
         (path "/4aa4a0cf-3721-431d-88e8-8afb2cf87302/e67f9728-ca0e-433d-883c-80e42a6fd80b"
-          (reference "#PWR0146") (unit 1)
+          (reference "#PWR01103") (unit 1)
         )
       )
@@
   (symbol (lib_id "capstone:SLG55021") (at 126.365 98.425 0) (unit 1)
     (in_bom yes) (on_board yes) (dnp no) (fields_autoplaced)
-    (property "Reference" "U13" (at 121.9709 84.455 0)
+    (property "Reference" "U1102" (at 121.9709 84.455 0)
       (effects (font (size 1.27 1.27)) (justify left))
     )
@@
       (project "high-power"
         (path "/4aa4a0cf-3721-431d-88e8-8afb2cf87302/e67f9728-ca0e-433d-883c-80e42a6fd80b"
-          (reference "U13") (unit 1)
+          (reference "U1102") (unit 1)
         )
       )
@@
   (symbol (lib_id "Device:C") (at 48.26 102.87 0) (unit 1)
     (in_bom yes) (on_board yes) (dnp no)
-    (property "Reference" "C149" (at 51.435 101.6 0)
+    (property "Reference" "C1101" (at 51.435 101.6 0)
       (effects (font (size 1.27 1.27)) (justify left))
     )
@@
       (project "high-power"
         (path "/4aa4a0cf-3721-431d-88e8-8afb2cf87302/e67f9728-ca0e-433d-883c-80e42a6fd80b"
-          (reference "C149") (unit 1)
+          (reference "C1101") (unit 1)
         )
       )
@@
         )
         (path "/4aa4a0cf-3721-431d-88e8-8afb2cf87302/e67f9728-ca0e-433d-883c-80e42a6fd80b"
-          (reference "R187") (unit 1)
+          (reference "R1104") (unit 1)
         )
       )
@@
   (symbol (lib_id "Device:R") (at 109.855 102.87 0) (unit 1)
     (in_bom yes) (on_board yes) (dnp no) (fields_autoplaced)
-    (property "Reference" "R185" (at 111.76 102.235 0)
+    (property "Reference" "R1102" (at 111.76 102.235 0)
       (effects (font (size 1.27 1.27)) (justify left))
     )
@@
       (project "high-power"
         (path "/4aa4a0cf-3721-431d-88e8-8afb2cf87302/e67f9728-ca0e-433d-883c-80e42a6fd80b"
-          (reference "R185") (unit 1)
+          (reference "R1102") (unit 1)
         )
       )
@@
         )
         (path "/4aa4a0cf-3721-431d-88e8-8afb2cf87302/e67f9728-ca0e-433d-883c-80e42a6fd80b"
-          (reference "Q38") (unit 1)
+          (reference "Q1102") (unit 1)
         )
       )
@@
         )
         (path "/4aa4a0cf-3721-431d-88e8-8afb2cf87302/e67f9728-ca0e-433d-883c-80e42a6fd80b"
-          (reference "TP11") (unit 1)
+          (reference "TP1101") (unit 1)
         )
       )
@@
   (symbol (lib_name "GND_1") (lib_id "power:GND") (at 120.015 109.22 0) (unit 1)
     (in_bom yes) (on_board yes) (dnp no) (fields_autoplaced)
-    (property "Reference" "#PWR0147" (at 120.015 115.57 0)
+    (property "Reference" "#PWR01104" (at 120.015 115.57 0)
       (effects (font (size 1.27 1.27)) hide)
     )
@@
       (project "high-power"
         (path "/4aa4a0cf-3721-431d-88e8-8afb2cf87302/e67f9728-ca0e-433d-883c-80e42a6fd80b"
-          (reference "#PWR0147") (unit 1)
+          (reference "#PWR01104") (unit 1)
         )
       )
@@
   (symbol (lib_id "Device:R") (at 60.96 102.87 0) (unit 1)
     (in_bom yes) (on_board yes) (dnp no) (fields_autoplaced)
-    (property "Reference" "R184" (at 62.865 102.235 0)
+    (property "Reference" "R1101" (at 62.865 102.235 0)
       (effects (font (size 1.27 1.27)) (justify left))
     )
@@
       (project "high-power"
         (path "/4aa4a0cf-3721-431d-88e8-8afb2cf87302/e67f9728-ca0e-433d-883c-80e42a6fd80b"
-          (reference "R184") (unit 1)
-        )
-      )
+          (reference "R1101") (unit 1)
+        )
+      )
