File: hardware/boards/low-power/digital_radio.kicad_sch (KiCad schematic)
At the start: 35 parts, among them J1 U.FL, U1 SX1262IMLTRT, U2 SKY13453-385LF, Y1 32 MHz

Commit message: Add footprints and models for LP board
Also completed rough layout for LP board to estimate board space usage.
Parts:
- C20: footprint Capacitor_SMD:C_0402_1005Metric -> Capacitor_SMD:C_0201_0603Metric
- J1: footprint Connector_PinSocket_2.54mm:PinSocket_1x05_P2.54mm_Vertical -> capstone:U.FL-R-SMT-1(60)
Changed lines of the file:
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@@
       (effects (font (size 1.27 1.27)) (justify right))
     )
-    (property "Footprint" "Capacitor_SMD:C_0402_1005Metric" (at 228.9048 84.455 0)
+    (property "Footprint" "Capacitor_SMD:C_0201_0603Metric" (at 228.9048 84.455 0)
       (effects (font (size 1.27 1.27)) hide)
     )
@@
       (effects (font (size 1.27 1.27)) (justify left))
     )
-    (property "Footprint" "Connector_PinSocket_2.54mm:PinSocket_1x05_P2.54mm_Vertical" (at 271.78 79.375 0)
-      (effects (font (size 1.27 1.27)) hide)
-    )
+    (property "Footprint" "capstone:U.FL-R-SMT-1(60)" (at 271.78 79.375 0)
+      (effects (font (size 1.27 1.27)) hide)
+    )

Commit message: Add initial changes after schematic review
Parts:
- C16: value 100n -> 10n
- renumbered R1 to R401
