File: hardware/boards/low-power/gps.kicad_sch (KiCad schematic)
At the start: 5 parts, among them U6 L80-R

Commit message: Add footprints and models for LP board
Also completed rough layout for LP board to estimate board space usage.
Parts:
- U6: footprint RF_GPS:Quectel_L80-R -> capstone:Quectel_L80-R
Changed lines of the file:
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@@
       (effects (font (size 1.27 1.27)) (justify left))
     )
-    (property "Footprint" "RF_GPS:Quectel_L80-R" (at 154.94 129.54 0)
+    (property "Footprint" "capstone:Quectel_L80-R" (at 154.94 129.54 0)
       (effects (font (size 1.27 1.27)) hide)
     )

Commit message: Add initial changes after schematic review
Parts:
- C44: value 2.2u -> 10u
- renumbered R25 to R201
Other:
- note added: "ONE 100n CAP FOR EACH PIN"
Changed lines of the file:
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@@
     (stroke (width 0) (type default))
+  )
+  (text "ONE 100n CAP\nFOR EACH PIN" (at 126.365 81.915 0)
+    (effects (font (size 1.27 1.27)) (justify left bottom))
   )
   (hierarchical_label "~{RESET}" (shape input) (at 121.92 111.76 180) (fields_autoplaced)
@@
         )
         (path "/71f6a5b4-1ac6-435b-9486-30b16ab86e62/a6608ad1-69a0-4d23-9644-6c2efafa5ff5"
-          (reference "#PWR07") (unit 1)
+          (reference "#PWR0202") (unit 1)
         )
       )
@@
       (effects (font (size 1.27 1.27)) (justify left))
     )
-    (property "Value" "2.2u" (at 144.145 91.44 0)
+    (property "Value" "10u" (at 144.145 91.44 0)
       (effects (font (size 1.27 1.27)) (justify left))
     )
@@
         )
         (path "/71f6a5b4-1ac6-435b-9486-30b16ab86e62/a6608ad1-69a0-4d23-9644-6c2efafa5ff5"
-          (reference "C3") (unit 1)
+          (reference "C203") (unit 1)
         )
       )
@@
         )
         (path "/71f6a5b4-1ac6-435b-9486-30b16ab86e62/a6608ad1-69a0-4d23-9644-6c2efafa5ff5"
-          (reference "#PWR06") (unit 1)
+          (reference "#PWR0201") (unit 1)
         )
       )
@@
         )
         (path "/71f6a5b4-1ac6-435b-9486-30b16ab86e62/a6608ad1-69a0-4d23-9644-6c2efafa5ff5"
-          (reference "C1") (unit 1)
+          (reference "C201") (unit 1)
         )
       )
@@
         )
         (path "/71f6a5b4-1ac6-435b-9486-30b16ab86e62/a6608ad1-69a0-4d23-9644-6c2efafa5ff5"
-          (reference "U1") (unit 1)
+          (reference "U201") (unit 1)
         )
       )
@@
   (symbol (lib_id "Device:R") (at 135.89 116.205 0) (unit 1)
     (in_bom yes) (on_board yes) (dnp no)
-    (property "Reference" "R25" (at 137.795 115.57 0)
+    (property "Reference" "R201" (at 137.795 115.57 0)
       (effects (font (size 1.27 1.27)) (justify left))
     )
@@
       (project "low-power"
         (path "/71f6a5b4-1ac6-435b-9486-30b16ab86e62/a6608ad1-69a0-4d23-9644-6c2efafa5ff5"
-          (reference "R25") (unit 1)
+          (reference "R201") (unit 1)
         )
       )
@@
         )
         (path "/71f6a5b4-1ac6-435b-9486-30b16ab86e62/a6608ad1-69a0-4d23-9644-6c2efafa5ff5"
-          (reference "C2") (unit 1)
-        )
-      )
+          (reference "C202") (unit 1)
+        )
+      )
