File: hardware/boards/low-power/low-power.kicad_sch (KiCad schematic)
At the start: 2 parts, among them J1 Conn_01x05_Pin, J2 Conn_01x32_Pin

Commit message: Add footprints and models for LP board
Also completed rough layout for LP board to estimate board space usage.
Parts:
- J1: footprint Connector_PinSocket_1.27mm:PinSocket_1x05_P1.27mm_Vertical -> Connector_JST:JST_GH_SM05B-GHS-TB_1x05-1MP_P1.25mm_Horizontal
- J2: footprint Connector_PinHeader_2.54mm:PinHeader_2x16_P2.54mm_Vertical -> Connector_PinHeader_1.27mm:PinHeader_2x16_P1.27mm_Vertical
Changed lines of the file:
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@@
       (effects (font (size 1.27 1.27)))
     )
-    (property "Footprint" "Connector_PinHeader_2.54mm:PinHeader_2x16_P2.54mm_Vertical" (at 32.385 121.92 0)
+    (property "Footprint" "Connector_PinHeader_1.27mm:PinHeader_2x16_P1.27mm_Vertical" (at 32.385 121.92 0)
       (effects (font (size 1.27 1.27)) hide)
     )
@@
       (effects (font (size 1.27 1.27)))
     )
-    (property "Footprint" "Connector_PinSocket_1.27mm:PinSocket_1x05_P1.27mm_Vertical" (at 32.385 53.975 0)
+    (property "Footprint" "Connector_JST:JST_GH_SM05B-GHS-TB_1x05-1MP_P1.25mm_Horizontal" (at 32.385 53.975 0)
       (effects (font (size 1.27 1.27)) hide)
     )

Commit message: Add initial changes after schematic review
Parts:
- renumbered J1 to J101, J2 to J102
Connections:
- net VIDEO_RX: now also J101.5 (Pin_5); no longer J101.4 (Pin_4)
- net VIDEO_TX: now also J101.4 (Pin_4); no longer J101.5 (Pin_5)
Changed lines of the file:
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@@
     (effects (font (size 1.27 1.27)) (justify right bottom))
   )
-  (label "VIDEO_TX" (at 50.8 59.055 180) (fields_autoplaced)
+  (label "VIDEO_RX" (at 50.8 59.055 180) (fields_autoplaced)
     (effects (font (size 1.27 1.27)) (justify right bottom))
   )
@@
     (effects (font (size 1.27 1.27)) (justify right bottom))
   )
-  (label "VIDEO_RX" (at 50.8 56.515 180) (fields_autoplaced)
+  (label "VIDEO_TX" (at 50.8 56.515 180) (fields_autoplaced)
     (effects (font (size 1.27 1.27)) (justify right bottom))
   )
@@
   (symbol (lib_id "power:GND") (at 40.005 163.83 0) (unit 1)
     (in_bom yes) (on_board yes) (dnp no) (fields_autoplaced)
-    (property "Reference" "#PWR04" (at 40.005 170.18 0)
+    (property "Reference" "#PWR0105" (at 40.005 170.18 0)
       (effects (font (size 1.27 1.27)) hide)
     )
@@
       (project "low-power"
         (path "/71f6a5b4-1ac6-435b-9486-30b16ab86e62"
-          (reference "#PWR04") (unit 1)
+          (reference "#PWR0105") (unit 1)
         )
       )
@@
   (symbol (lib_id "power:+BATT") (at 40.259 47.625 0) (unit 1)
     (in_bom yes) (on_board yes) (dnp no)
-    (property "Reference" "#PWR05" (at 40.259 51.435 0)
+    (property "Reference" "#PWR0106" (at 40.259 51.435 0)
       (effects (font (size 1.27 1.27)) hide)
     )
@@
       (project "low-power"
         (path "/71f6a5b4-1ac6-435b-9486-30b16ab86e62"
-          (reference "#PWR05") (unit 1)
+          (reference "#PWR0106") (unit 1)
         )
         (path "/71f6a5b4-1ac6-435b-9486-30b16ab86e62/e8b4c09d-dc7e-4556-902a-6f0fed733097"
@@
   (symbol (lib_id "power:GND") (at 40.005 63.119 0) (unit 1)
     (in_bom yes) (on_board yes) (dnp no) (fields_autoplaced)
-    (property "Reference" "#PWR03" (at 40.005 69.469 0)
+    (property "Reference" "#PWR0104" (at 40.005 69.469 0)
       (effects (font (size 1.27 1.27)) hide)
     )
@@
       (project "low-power"
         (path "/71f6a5b4-1ac6-435b-9486-30b16ab86e62"
-          (reference "#PWR03") (unit 1)
+          (reference "#PWR0104") (unit 1)
         )
       )
@@
   (symbol (lib_id "power:+3.3V") (at 39.37 119.38 270) (unit 1)
     (in_bom yes) (on_board yes) (dnp no)
-    (property "Reference" "#PWR01" (at 35.56 119.38 0)
+    (property "Reference" "#PWR0101" (at 35.56 119.38 0)
       (effects (font (size 1.27 1.27)) hide)
     )
@@
       (project "low-power"
         (path "/71f6a5b4-1ac6-435b-9486-30b16ab86e62"
-          (reference "#PWR01") (unit 1)
+          (reference "#PWR0101") (unit 1)
         )
       )
@@
   (symbol (lib_id "power:+5V") (at 39.37 121.92 270) (unit 1)
     (in_bom yes) (on_board yes) (dnp no)
-    (property "Reference" "#PWR02" (at 35.56 121.92 0)
+    (property "Reference" "#PWR0102" (at 35.56 121.92 0)
       (effects (font (size 1.27 1.27)) hide)
     )
@@
       (project "low-power"
         (path "/71f6a5b4-1ac6-435b-9486-30b16ab86e62"
-          (reference "#PWR02") (unit 1)
+          (reference "#PWR0102") (unit 1)
         )
       )
@@
   (symbol (lib_id "power:+BATT") (at 39.37 124.46 270) (unit 1)
     (in_bom yes) (on_board yes) (dnp no) (fields_autoplaced)
-    (property "Reference" "#PWR063" (at 35.56 124.46 0)
+    (property "Reference" "#PWR0103" (at 35.56 124.46 0)
       (effects (font (size 1.27 1.27)) hide)
     )
@@
       (project "low-power"
         (path "/71f6a5b4-1ac6-435b-9486-30b16ab86e62"
-          (reference "#PWR063") (unit 1)
+          (reference "#PWR0103") (unit 1)
         )
       )
@@
   (symbol (lib_id "Connector:Conn_01x32_Pin") (at 32.385 121.92 0) (unit 1)
     (in_bom yes) (on_board yes) (dnp no) (fields_autoplaced)
-    (property "Reference" "J2" (at 33.02 80.01 0)
+    (property "Reference" "J102" (at 33.02 80.01 0)
       (effects (font (size 1.27 1.27)))
     )
@@
       (project "low-power"
         (path "/71f6a5b4-1ac6-435b-9486-30b16ab86e62"
-          (reference "J2") (unit 1)
+          (reference "J102") (unit 1)
         )
       )
@@
   (symbol (lib_id "Connector:Conn_01x05_Pin") (at 32.385 53.975 0) (unit 1)
     (in_bom yes) (on_board yes) (dnp no)
-    (property "Reference" "J1" (at 32.639 46.101 0)
+    (property "Reference" "J101" (at 32.639 46.101 0)
       (effects (font (size 1.27 1.27)))
     )
@@
       (project "low-power"
         (path "/71f6a5b4-1ac6-435b-9486-30b16ab86e62"
-          (reference "J1") (unit 1)
-        )
-      )
+          (reference "J101") (unit 1)
+        )
+      )
