File: hardware/boards/low-power/usb.kicad_sch (KiCad schematic)
At the start: 9 parts

Commit message: Add footprints and models for LP board
Also completed rough layout for LP board to estimate board space usage.
Parts:
- J?: footprint Connector_PinHeader_2.54mm:PinHeader_2x16_P2.54mm_Vertical -> Connector_USB:USB_C_Receptacle_G-Switch_GT-USB-7010ASV
Changed lines of the file:
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@@
       (effects (font (size 1.27 1.27)))
     )
-    (property "Footprint" "Connector_PinHeader_2.54mm:PinHeader_2x16_P2.54mm_Vertical" (at 74.295 93.98 0)
+    (property "Footprint" "Connector_USB:USB_C_Receptacle_G-Switch_GT-USB-7010ASV" (at 74.295 93.98 0)
       (effects (font (size 1.27 1.27)) hide)
     )

Commit message: Add initial changes after schematic review
Parts:
- added R1002, R1003, R1004, R1005, R1006, R1007, R1008, R1009: 0R, symbol Device:R
- renumbered C63 to C1001, D2 to D1001
Connections:
- net GND: now also R1003.2, R1005.2, R1007.2, R1009.2; no longer U?.1 (VBUS_MIN)
- net USBPD_3V3: now also R1002.1, R1004.1, R1006.1, R1008.1; no longer U?.2 (VBUS_MAX), U?.5 (ISINK_COARSE), U?.6 (ISINK_FINE)
- new net: R1006.2, R1007.1, U?.5 (ISINK_COARSE)
- new net: R1002.2, R1003.1, U?.1 (VBUS_MIN)
- new net: R1004.2, R1005.1, U?.2 (VBUS_MAX)
- new net: R1008.2, R1009.1, U?.6 (ISINK_FINE)
