File: hardware/boards/low-power/video_radio.kicad_sch (KiCad schematic)
At the start: 4 parts, among them J5 U.FL, U11 TX5813

Commit message: Add initial changes after schematic review
Parts:
- C61, C62: footprint Capacitor_SMD:C_0805_2012Metric -> Capacitor_SMD:C_0603_1608Metric
Changed lines of the file:
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@@
       (effects (font (size 1.27 1.27)) (justify left))
     )
-    (property "Footprint" "Capacitor_SMD:C_0805_2012Metric" (at 169.2148 107.315 0)
+    (property "Footprint" "Capacitor_SMD:C_0603_1608Metric" (at 169.2148 107.315 0)
       (effects (font (size 1.27 1.27)) hide)
     )
@@
         )
         (path "/71f6a5b4-1ac6-435b-9486-30b16ab86e62/2c81f013-3430-433c-abe0-42fcceae4b74"
-          (reference "C5") (unit 1)
+          (reference "C302") (unit 1)
         )
       )
@@
         )
         (path "/71f6a5b4-1ac6-435b-9486-30b16ab86e62/2c81f013-3430-433c-abe0-42fcceae4b74"
-          (reference "#PWR08") (unit 1)
+          (reference "#PWR0301") (unit 1)
         )
       )
@@
         )
         (path "/71f6a5b4-1ac6-435b-9486-30b16ab86e62/2c81f013-3430-433c-abe0-42fcceae4b74"
-          (reference "J3") (unit 1)
+          (reference "J301") (unit 1)
         )
       )
@@
         )
         (path "/71f6a5b4-1ac6-435b-9486-30b16ab86e62/2c81f013-3430-433c-abe0-42fcceae4b74"
-          (reference "#PWR09") (unit 1)
+          (reference "#PWR0302") (unit 1)
         )
       )
@@
         )
         (path "/71f6a5b4-1ac6-435b-9486-30b16ab86e62/2c81f013-3430-433c-abe0-42fcceae4b74"
-          (reference "U2") (unit 1)
+          (reference "U301") (unit 1)
         )
       )
@@
       (effects (font (size 1.27 1.27)))
     )
-    (property "Footprint" "Capacitor_SMD:C_0805_2012Metric" (at 129.54 101.9048 0)
+    (property "Footprint" "Capacitor_SMD:C_0603_1608Metric" (at 129.54 101.9048 0)
       (effects (font (size 1.27 1.27)) hide)
     )
@@
         )
         (path "/71f6a5b4-1ac6-435b-9486-30b16ab86e62/2c81f013-3430-433c-abe0-42fcceae4b74"
-          (reference "C4") (unit 1)
+          (reference "C301") (unit 1)
         )
       )
