File: hardware/boards/ground-station/radio.kicad_sch (KiCad schematic)
At the start: 54 parts, among them J1 U.FL, J3 Conn_Coaxial, J5 U.FL, U1 SX1262IMLTRT, U2 SKY13453-385LF, U201 SW-GPS01, U202 RX5808, Y1 32 MHz

Commit message: base station layout review
Parts:
- added C3: 100n, Capacitor_SMD:C_0201_0603Metric, symbol Device:C
- added R208: 0, Resistor_SMD:R_0402_1005Metric, symbol Device:R_Small
Connections:
- net +3V3: now also C3.1
- net GND: now also C3.2
- net VIDEO_OUT: now also R208.1; no longer J3.1 (In)
- new net: J3.1 (In), R208.2
Changed lines of the file:
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@@
   (junction (at 62.865 76.835) (diameter 0) (color 0 0 0 0)
+  )
+  (junction (at 33.655 20.955) (diameter 0) (color 0 0 0 0)
   )
   (junction (at 97.155 176.53) (diameter 0) (color 0 0 0 0)
@@
     (stroke (width 0) (type default))
   )
+  (wire (pts (xy 33.655 29.845) (xy 33.655 31.115))
+    (stroke (width 0) (type default))
+  )
   (wire (pts (xy 97.79 79.375) (xy 85.725 79.375))
     (stroke (width 0) (type default))
@@
     (stroke (width 0) (type default))
   )
-  (wire (pts (xy 45.085 19.685) (xy 45.085 20.955))
+  (wire (pts (xy 33.655 20.32) (xy 33.655 20.955))
     (stroke (width 0) (type default))
   )
@@
     (stroke (width 0) (type default))
   )
+  (wire (pts (xy 33.655 31.115) (xy 45.085 31.115))
+    (stroke (width 0) (type default))
+  )
+  (wire (pts (xy 33.655 20.955) (xy 45.085 20.955))
+    (stroke (width 0) (type default))
+  )
   (wire (pts (xy 61.595 29.845) (xy 64.135 29.845))
     (stroke (width 0) (type default))
@@
     (stroke (width 0) (type default))
   )
-  (wire (pts (xy 118.11 161.29) (xy 100.33 161.29))
+  (wire (pts (xy 118.11 161.29) (xy 111.76 161.29))
     (stroke (width 0) (type default))
   )
@@
   )
   (wire (pts (xy 100.965 46.355) (xy 111.125 46.355))
+    (stroke (width 0) (type default))
+  )
+  (wire (pts (xy 33.655 22.225) (xy 33.655 20.955))
     (stroke (width 0) (type default))
   )
@@
   )
   (wire (pts (xy 234.95 29.21) (xy 245.11 29.21))
+    (stroke (width 0) (type default))
+  )
+  (wire (pts (xy 106.68 161.29) (xy 100.33 161.29))
     (stroke (width 0) (type default))
   )
@@
     )
   )
+  (symbol (lib_id "Device:R_Small") (at 109.22 161.29 90) (unit 1)
+    (in_bom yes) (on_board yes) (dnp yes)
+    (property "Reference" "R208" (at 105.41 160.02 90)
+      (effects (font (size 1.27 1.27)))
+    )
+    (property "Value" "0" (at 111.76 160.02 90)
+      (effects (font (size 1.27 1.27)))
+    )
+    (property "Footprint" "Resistor_SMD:R_0402_1005Metric" (at 109.22 161.29 0)
+      (effects (font (size 1.27 1.27)) hide)
+    )
+    (property "Datasheet" "~" (at 109.22 161.29 0)
+      (effects (font (size 1.27 1.27)) hide)
+    )
+    (pin "1")
+    (pin "2")
+    (instances
+      (project "ground-station"
+        (path "/ce329892-de08-4d39-b253-15f3aaf1c085/37a6bbaf-9821-4b58-bc66-fc0453299811"
+          (reference "R208") (unit 1)
+        )
+      )
+    )
+  )
   (symbol (lib_id "capstone:RX5808") (at 63.5 172.72 0) (unit 1)
     (in_bom yes) (on_board yes) (dnp no) (fields_autoplaced)
@@
     )
   )
-  (symbol (lib_id "power:+3V3") (at 45.085 19.685 0) (unit 1)
-    (in_bom yes) (on_board yes) (dnp no)
-    (property "Reference" "#PWR0401" (at 45.085 23.495 0)
-      (effects (font (size 1.27 1.27)) hide)
-    )
-    (property "Value" "+3V3" (at 45.085 15.875 0)
-      (effects (font (size 1.27 1.27)))
-    )
-    (property "Footprint" "" (at 45.085 19.685 0)
-      (effects (font (size 1.27 1.27)) hide)
-    )
-    (property "Datasheet" "" (at 45.085 19.685 0)
+  (symbol (lib_id "power:+3V3") (at 33.655 20.32 0) (unit 1)
+    (in_bom yes) (on_board yes) (dnp no)
+    (property "Reference" "#PWR0401" (at 33.655 24.13 0)
+      (effects (font (size 1.27 1.27)) hide)
+    )
+    (property "Value" "+3V3" (at 33.655 16.51 0)
+      (effects (font (size 1.27 1.27)))
+    )
+    (property "Footprint" "" (at 33.655 20.32 0)
+      (effects (font (size 1.27 1.27)) hide)
+    )
+    (property "Datasheet" "" (at 33.655 20.32 0)
       (effects (font (size 1.27 1.27)) hide)
     )
@@
         )
       )
+    )
+  )
+  (symbol (lib_id "Device:C") (at 33.655 26.035 0) (unit 1)
+    (in_bom yes) (on_board yes) (dnp no)
+    (property "Reference" "C3" (at 36.195 24.765 0)
+      (effects (font (size 1.27 1.27)) (justify left))
+    )
+    (property "Value" "100n" (at 36.195 27.305 0)
+      (effects (font (size 1.27 1.27)) (justify left))
+    )
+    (property "Footprint" "Capacitor_SMD:C_0201_0603Metric" (at 34.6202 29.845 0)
+      (effects (font (size 1.27 1.27)) hide)
+    )
+    (property "Datasheet" "~" (at 33.655 26.035 0)
+      (effects (font (size 1.27 1.27)) hide)
+    )
+    (pin "1")
+    (pin "2")
+    (instances
+      (project "low-power"
+        (path "/71f6a5b4-1ac6-435b-9486-30b16ab86e62"
+          (reference "C3") (unit 1)
+        )
+        (path "/71f6a5b4-1ac6-435b-9486-30b16ab86e62/9ba2378d-16cf-4aed-809c-215b19eeadaa"
+          (reference "C402") (unit 1)
+        )
+      )
+      (project "ground-station"
+        (path "/ce329892-de08-4d39-b253-15f3aaf1c085/37a6bbaf-9821-4b58-bc66-fc0453299811"
+          (reference "C231") (unit 1)
+        )
+      )
